File: src/kicad-new/ardupi.kicad_sch (KiCad schematic)
At the start: 60 parts, among them J1 Conn_01x02, J10 Conn_01x04, J11 TSW-108-08-L-T-RA, J2 Conn_01x10, J3 Conn_01x05, J4 Conn_01x04, J5 GPIO_CONNECTOR, J6 Conn_01x05, J7 Conn_01x06, J8 Conn_01x04, J9 Conn_01x02, U1 CAT24C256, U2 ULN2803ADW, U3 PCA9685BS, U4 ADS1115IRUGR, U5 MPU-9250, U6 BMP280

Commit message: Basic pcb layout
Parts:
- removed BT1: Battery, symbol Device:Battery
- removed C1: 100n, symbol Device:C_Small
- removed J1: Conn_01x02, Connector_JST:JST_EH_B2B-EH-A_1x02_P2.50mm_Vertical, symbol ardupi:Conn_01x02
- removed J5: GPIO_CONNECTOR, lib:PinSocket_2x20_P2.54mm_Vertical_Centered_Anchor, symbol Connector_Generic:Conn_02x20_Odd_Even
- removed JP1: ID_WP, symbol Jumper:SolderJumper_2_Open
- removed R1, R2: 3.9k, symbol Device:R_Small
- added C9: 100n, symbol Device:C_Small
- added J1: GPIO, Connector_PinSocket_2.54mm:PinSocket_2x20_P2.54mm_Vertical, symbol Connector_Generic:Conn_02x20_Odd_Even
- added JP2: ID_WP, symbol Jumper:SolderJumper_2_Open
- added R21, R22: 3.9k, symbol Device:R_Small
Connections:
- net +3V3: now also U1.8 (VCC), C9.2, J1.1 (Pin_1), J1.17 (Pin_17), JP2.2 (B), R21.2, R22.1
- net +5V: now also J1.2 (Pin_2), J1.4 (Pin_4)
- net BUZZER: now also J1.32 (Pin_32)
- net GND: now also U1.4 (VSS), C9.1, J1.14 (Pin_14), J1.20 (Pin_20), J1.25 (Pin_25), J1.30 (Pin_30), J1.34 (Pin_34), J1.39 (Pin_39), J1.6 (Pin_6), J1.9 (Pin_9)
- net GPIO14_TXD0: now also J1.8 (Pin_8)
- net GPIO15_RXD0: now also J1.10 (Pin_10)
- net GPIO18_GEN1: now also J1.12 (Pin_12)
- net GPIO23: now also J1.16 (Pin_16)
- net GPIO24: now also J1.18 (Pin_18)
- net GPIO25_GEN6: now also J1.22 (Pin_22)
- net ID_SCL: now also U1.6 (SCL), U1.7 (WP), J1.28 (Pin_28), JP2.1 (A), R22.2
- net ID_SDA: now also U1.5 (SDA), J1.27 (Pin_27), R21.1
- net LED1: now also J1.13 (Pin_13)
- net LED2: now also J1.15 (Pin_15)
- net LED3: now also J1.7 (Pin_7)
- net RC1: now also J1.29 (Pin_29)
- net RC2: now also J1.31 (Pin_31)
- net RC3: now also J1.33 (Pin_33)
- net RC4: now also J1.35 (Pin_35)
- net RC5: now also J1.37 (Pin_37)
- net RC6: now also J1.40 (Pin_40)
- net RC7: now also J1.38 (Pin_38)
- net RC8: now also J1.36 (Pin_36)
- net SCL1: now also J1.5 (Pin_5)
- net SDA1: now also J1.3 (Pin_3)
- net SPI_CE0_N: now also J1.24 (Pin_24)
- net SPI_CE1_N: now also J1.26 (Pin_26)
- net SPI_MISO: now also J1.21 (Pin_21)
- net SPI_MOSI: now also J1.19 (Pin_19)
- net SPI_SCLK: now also J1.23 (Pin_23)
- net SRVO_EN: now also J1.11 (Pin_11)
Other:
- title: ArduPi -> (none)
- moved on the sheet: C_PCA1, J11, R3, R4, R5, U1, U3
