File: src/hardware/ardupi-pca9685.kicad_sch (KiCad schematic)
At the start: 43 parts, among them J1 Conn_01x05, J2 Conn_01x06, J3 RPI-4B-Header, J5 Conn_01x02, J6 Conn_01x04, J7 Conn_01x04, J8 Conn_01x05, J9 Conn_01x10, M1 NEO-M8Q-01A, U1 ULN2803ADWR, U2 CAT24C32WI-GT3, U3 ADS1115IDGSR, U4 RFM95W-915S2, U5 MPU-9250, U7 BMP280

Commit message: removed pca9685, fall back to adafruit module. As per original OBAL footprint / design
Parts:
- removed J?: Conn_01x06, Connector_JST:JST_EH_B6B-EH-A_1x06_P2.50mm_Vertical, symbol Connector_Generic:Conn_01x06
- added C_PCA1: 10uF, Capacitor_SMD:CP_Elec_8x5.4, symbol Device:C_Polarized
- added J4: PWM_Header, Ardupi:PWM_Header, symbol ArduPi:PWM_Header
- added R1, R10, R5, R6, R8: 10k, Resistor_SMD:R_0402_1005Metric, symbol Device:R_Small
- added R16, R17, R18, R19, R20, R21, R22, R23: 220 Ω, Resistor_SMD:R_0402_1005Metric, symbol Device:R_Small
- added R2, R3, R4: 10K, Resistor_SMD:R_0402_1005Metric, symbol Device:R_Small
- added SJ1, SJ2, SJ3, SJ4, SJ5, SJ6: SolderJumper-Open_Pad, Ardupi:SolderJumper-Open_Pad, symbol ArduPi:SolderJumper-Open_Pad
- added U6: PCA9685PW, Ardupi:PCA9685PW, symbol ArduPi:PCA9685PW
- added U8: MPU-9250, Ardupi:MPU-9250, symbol ArduPi:MPU-9250
Connections:
- net +5V: now also C_PCA1.1, R10.1, R8.1, SJ1.1, SJ2.1, SJ3.1, SJ4.1, SJ5.1, SJ6.1, U6.28 (VDD)
- net GND: now also C_PCA1.2, J4.12, J4.15, J4.18, J4.21, J4.24, J4.3, J4.6, J4.9, R1.2, R2.2, R3.2, R4.2, R5.2, R6.2, U6.14 (VSS), U6.25 (EXTCLK)
- net PCA_EN: now also U6.23 (OE)
- net SCL1: now also R8.2, U6.26 (SCL)
- net SDA1: now also R10.2, U6.27 (SDA)
- net V_EXT: now also J4.11, J4.14, J4.17, J4.2, J4.20, J4.23, J4.5, J4.8
- new net: J4.13, R23.2
- new net: R1.1, SJ1.2, U6.1 (A0)
- new net: R3.1, SJ3.2, U6.3 (A2)
- new net: J4.4, R17.1
- new net: J4.10, R19.1
- new net: J4.16, R22.2
- new net: R6.1, SJ6.2, U6.24 (A5)
- new net: J4.1, R16.1
- new net: J4.19, R21.2
- new net: J4.22, R20.2
- new net: J4.7, R18.1
- new net: R2.1, SJ2.2, U6.2 (A1)
- new net: R4.1, SJ4.2, U6.4 (A3)
- new net: R5.1, SJ5.2, U6.5 (A4)
- new net PWM1: R16.2, U6.6 (LED0)
- new net PWM10: U6.16 (LED9)
- new net PWM11: U6.17 (LED10)
- new net PWM12: U6.18 (LED11)
- new net PWM13: U6.19 (LED12)
- new net PWM14: U6.20 (LED13)
- new net PWM15: U6.21 (LED14)
- new net PWM16: U6.22 (LED15)
- new net PWM2: R17.2, U6.7 (LED1)
- new net PWM3: R18.2, U6.8 (LED2)
- new net PWM4: R19.2, U6.9 (LED3)
- new net PWM5: R23.1, U6.10 (LED4)
- new net PWM6: R22.1, U6.11 (LED5)
- new net PWM7: R21.1, U6.12 (LED6)
- new net PWM8: R20.1, U6.13 (LED7)
- new net PWM9: U6.15 (LED8)
Other:
- note added: "PWM Header"
- moved on the sheet: C2, C3, C4, C5, C6, C7, C8, J1, J2, J5, J6, J7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
